File: antenna.sch (KiCad schematic (older format))
At the start: 8 parts

Commit message: Added missing 2.2uF cap to LTC4063 LDO output, normalized capacitor values to micro and pico, removed units from component values
Parts:
- C13: value 1.5pF -> 1.5p
- C5: value 2.2nF -> 2200p
- C6: value 2.2pF -> 2.2p
- C8: value 1pF -> 1p
- L1: value 4.7nH -> 4.7n
- L2: value 10nH -> 10n
- L3: value 3.3nH -> 3.3n
Changed lines of the file:
@@
 P 3300 2500
 F 0 "L1" V 3350 2450 50  0000 C CNN
-F 1 "4.7nH" V 3250 2400 50  0000 C CNN
+F 1 "4.7n" V 3250 2400 50  0000 C CNN
 F 2 "SMD_Packages:SMD-0402" H 3300 2500 60  0001 C CNN
 F 3 "~" H 3300 2500 60  0000 C CNN
@@
 P 3300 3100
 F 0 "L2" V 3350 3050 50  0000 C CNN
-F 1 "10nH" V 3250 3000 50  0000 C CNN
+F 1 "10n" V 3250 3000 50  0000 C CNN
 F 2 "SMD_Packages:SMD-0402" H 3300 3100 60  0001 C CNN
 F 3 "~" H 3300 3100 60  0000 C CNN
@@
 P 3300 3650
 F 0 "C5" H 3350 3750 40  0000 L CNN
-F 1 "2.2nF" H 3350 3550 40  0000 L CNN
+F 1 "2200p" H 3350 3550 40  0000 L CNN
 F 2 "SMD_Packages:SMD-0402" H 3338 3500 30  0001 C CNN
 F 3 "" H 3300 3650 60  0000 C CNN
@@
 P 3650 2250
 F 0 "C6" V 3500 2200 40  0000 L CNN
-F 1 "2.2pF" V 3800 2200 40  0000 L CNN
+F 1 "2.2p" V 3800 2200 40  0000 L CNN
 F 2 "SMD_Packages:SMD-0402" H 3688 2100 30  0001 C CNN
 F 3 "" H 3650 2250 60  0000 C CNN
@@
 P 3950 2600
 F 0 "C8" H 3850 2500 40  0000 L CNN
-F 1 "1pF" H 3900 2700 40  0000 R CNN
+F 1 "1p" H 3900 2700 40  0000 R CNN
 F 2 "SMD_Packages:SMD-0402" H 3988 2450 30  0001 C CNN
 F 3 "" H 3950 2600 60  0000 C CNN
@@
 P 4350 2250
 F 0 "L3" H 4350 2350 50  0000 C CNN
-F 1 "3.3nH" H 4350 2200 50  0000 C CNN
+F 1 "3.3n" H 4350 2200 50  0000 C CNN
 F 2 "SMD_Packages:SMD-0402" H 4350 2250 60  0001 C CNN
 F 3 "~" H 4350 2250 60  0000 C CNN
@@
 P 4750 2600
 F 0 "C13" H 4650 2500 40  0000 L CNN
-F 1 "1.5pF" H 4700 2700 40  0000 R CNN
+F 1 "1.5p" H 4700 2700 40  0000 R CNN
 F 2 "SMD_Packages:SMD-0402" H 4788 2450 30  0001 C CNN
 F 3 "" H 4750 2600 60  0000 C CNN

Commit message: Fixed footprints for MCU and USB-UART, added testpoints
Changed lines of the file:
@@
 EESchema Schematic File Version 2
+LIBS:watch-rescue
 LIBS:power
 LIBS:device
@@
 	3300 3350 3300 3450
 $Comp
-L GND #PWR025
+L GND-RESCUE-watch #PWR025
 U 1 1 5462B35F
 P 3300 3950
+AR Path="/5462B35F" Ref="#PWR025"  Part="1"
+AR Path="/5462AC04/5462B35F" Ref="#PWR025"  Part="1"
 F 0 "#PWR025" H 3300 3950 30  0001 C CNN
 F 1 "GND" H 3300 3880 30  0001 C CNN
@@
 Connection ~ 3300 2250
 $Comp
-L GND #PWR026
+L GND-RESCUE-watch #PWR026
 U 1 1 5462B38F
 P 3950 3000
+AR Path="/5462B38F" Ref="#PWR026"  Part="1"
+AR Path="/5462AC04/5462B38F" Ref="#PWR026"  Part="1"
 F 0 "#PWR026" H 3950 3000 30  0001 C CNN
 F 1 "GND" H 3950 2930 30  0001 C CNN
@@
 $EndComp
 $Comp
-L GND #PWR027
+L GND-RESCUE-watch #PWR027
 U 1 1 5462B395
 P 4750 3000
+AR Path="/5462B395" Ref="#PWR027"  Part="1"
+AR Path="/5462AC04/5462B395" Ref="#PWR027"  Part="1"
 F 0 "#PWR027" H 4750 3000 30  0001 C CNN
 F 1 "GND" H 4750 2930 30  0001 C CNN
