File: display.sch (KiCad schematic (older format))
At the start: 11 parts, among them U2 ER-OLED015-1, U8 MMBD4148SE

Commit message: Added missing 2.2uF cap to LTC4063 LDO output, normalized capacitor values to micro and pico, removed units from component values
Parts:
- C18, C19: value 100n -> 0.1u
Changed lines of the file:
@@
 P 3250 2300
 F 0 "C19" H 3250 2400 40  0000 L CNN
-F 1 "100n" H 3256 2215 40  0000 L CNN
+F 1 "0.1u" H 3256 2215 40  0000 L CNN
 F 2 "SMD_Packages:SMD-0603" H 3288 2150 30  0001 C CNN
 F 3 "" H 3250 2300 60  0000 C CNN
@@
 P 3200 3500
 F 0 "C18" H 3200 3600 40  0000 L CNN
-F 1 "100n" H 3206 3415 40  0000 L CNN
+F 1 "0.1u" H 3206 3415 40  0000 L CNN
 F 2 "SMD_Packages:SMD-0603" H 3238 3350 30  0001 C CNN
 F 3 "" H 3200 3500 60  0000 C CNN

Commit message: Fixed footprints for MCU and USB-UART, added testpoints
Changed lines of the file:
@@
 EESchema Schematic File Version 2
+LIBS:watch-rescue
 LIBS:power
 LIBS:device
@@
 $EndComp
 $Comp
-L GND #PWR028
+L GND-RESCUE-watch #PWR028
 U 1 1 546AB6EA
 P 3050 2600
+AR Path="/546AB6EA" Ref="#PWR028"  Part="1"
+AR Path="/546AB3F2/546AB6EA" Ref="#PWR028"  Part="1"
 F 0 "#PWR028" H 3050 2600 30  0001 C CNN
 F 1 "GND" H 3050 2530 30  0001 C CNN
@@
 $EndComp
 $Comp
-L GND #PWR029
+L GND-RESCUE-watch #PWR029
 U 1 1 546AB806
 P 3600 2750
+AR Path="/546AB806" Ref="#PWR029"  Part="1"
+AR Path="/546AB3F2/546AB806" Ref="#PWR029"  Part="1"
 F 0 "#PWR029" H 3600 2750 30  0001 C CNN
 F 1 "GND" H 3600 2680 30  0001 C CNN
@@
 	3200 3050 3200 3300
 $Comp
-L GND #PWR031
+L GND-RESCUE-watch #PWR031
 U 1 1 546AF672
 P 2200 3900
+AR Path="/546AF672" Ref="#PWR031"  Part="1"
+AR Path="/546AB3F2/546AF672" Ref="#PWR031"  Part="1"
 F 0 "#PWR031" H 2200 3900 30  0001 C CNN
 F 1 "GND" H 2200 3830 30  0001 C CNN
@@
 Connection ~ 4350 4300
 $Comp
-L GND #PWR033
+L GND-RESCUE-watch #PWR033
 U 1 1 546B06EC
 P 4350 4550
+AR Path="/546B06EC" Ref="#PWR033"  Part="1"
+AR Path="/546AB3F2/546B06EC" Ref="#PWR033"  Part="1"
 F 0 "#PWR033" H 4350 4550 30  0001 C CNN
 F 1 "GND" H 4350 4480 30  0001 C CNN
@@
 	4100 4400 4100 4550
 $Comp
-L GND #PWR034
+L GND-RESCUE-watch #PWR034
 U 1 1 546B0891
 P 4100 4550
+AR Path="/546B0891" Ref="#PWR034"  Part="1"
+AR Path="/546AB3F2/546B0891" Ref="#PWR034"  Part="1"
 F 0 "#PWR034" H 4100 4550 30  0001 C CNN
 F 1 "GND" H 4100 4480 30  0001 C CNN
@@
 $EndComp
 $Comp
-L GND #PWR035
+L GND-RESCUE-watch #PWR035
 U 1 1 546B0B8B
 P 4100 3550
+AR Path="/546B0B8B" Ref="#PWR035"  Part="1"
+AR Path="/546AB3F2/546B0B8B" Ref="#PWR035"  Part="1"
 F 0 "#PWR035" H 4100 3550 30  0001 C CNN
 F 1 "GND" H 4100 3480 30  0001 C CNN
@@
 Connection ~ 5850 4100
 $Comp
-L GND #PWR036
+L GND-RESCUE-watch #PWR036
 U 1 1 546B0F6A
 P 5850 4550
+AR Path="/546B0F6A" Ref="#PWR036"  Part="1"
+AR Path="/546AB3F2/546B0F6A" Ref="#PWR036"  Part="1"
 F 0 "#PWR036" H 5850 4550 30  0001 C CNN
 F 1 "GND" H 5850 4480 30  0001 C CNN
@@
 NoConn ~ 5750 2700
 $Comp
-L GND #PWR037
+L GND-RESCUE-watch #PWR037
 U 1 1 546B27DB
 P 5850 3600
+AR Path="/546B27DB" Ref="#PWR037"  Part="1"
+AR Path="/546AB3F2/546B27DB" Ref="#PWR037"  Part="1"
 F 0 "#PWR037" H 5850 3600 30  0001 C CNN
 F 1 "GND" H 5850 3530 30  0001 C CNN
